File: pcb/dak-base-station.kicad_pcb (KiCad board)
At the start: 2 copper layers, 94 x 76.2 mm, 6 parts, among them J1 433 mHz Receiver, J2 433 mHz Transmitter, J3 DHT11_Breakout, U1 ESP32-OLED

Commit message: PCB!
Parts:
- J1: footprint Connector_PinSocket_2.54mm:PinSocket_1x04_P2.54mm_Vertical -> 1-My Parts:433Receiver
- moved J2 34.8 mm to (105.7, 71.9), turned to 0 degrees
- moved J3 34.0 mm to (89.2, 47.0), turned to 90 degrees
- moved H2 8.98 mm to (109.2, 106.7)
- moved H1 1.80 mm to (38.1, 45.7)
Connections:
- U1 pad 15: Net-(J3-Pad2) -> Net-(J2-Pad3)
- U1 pad 18: Net-(J2-Pad3) -> Net-(J3-Pad2)
Routing:
- net (no net): track 0.00 -> 40.6 mm, vias 0 -> 1
- net Net-(J1-Pad1): track 204.1 -> 187.9 mm
- net Net-(J3-Pad2): track 27.0 -> 14.5 mm
- net Net-(J2-Pad3): track 16.6 -> 20.1 mm
- net Net-(J2-Pad1): track 63.3 -> 66.7 mm
Other:
- board size 94 x 76.2 mm -> 87.6 x 76.2 mm
- board text added: "DAK 433 mHz Base"
- board text added: "JP2-1"
