File: pcb/dak-base-station.sch (KiCad schematic (older format))
At the start: 6 parts, among them J1 433 mHz Receiver, J2 433 mHz Transmitter, J3 DHT11_Breakout, U1 ESP32-OLED

Commit message: PCB!
Parts:
- J1: footprint Connector_PinSocket_2.54mm:PinSocket_1x04_P2.54mm_Vertical -> 1-My Parts:433Receiver
Connections:
- wire segments 29 -> 25
Changed lines of the file:
@@
 F 0 "J1" V 7100 5150 50  0000 C CNN
 F 1 "433 mHz Receiver" V 7000 5050 50  0000 C CNN
-F 2 "Connector_PinSocket_2.54mm:PinSocket_1x04_P2.54mm_Vertical" H 7400 5350 50  0001 C CNN
+F 2 "1-My Parts:433Receiver" H 7400 5350 50  0001 C CNN
 F 3 "~" H 7400 5350 50  0001 C CNN
 	1    7400 5350
@@
 L 1-My~Parts:433_mHz_Transmitter J2
 U 1 1 5DA27D0A
-P 7550 2800
-F 0 "J2" V 7400 3050 50  0000 C CNN
-F 1 "433 mHz Transmitter" V 7300 3100 50  0000 C CNN
-F 2 "Connector_PinSocket_2.54mm:PinSocket_1x03_P2.54mm_Vertical" H 7550 2800 50  0001 C CNN
-F 3 "~" H 7550 2800 50  0001 C CNN
-	1    7550 2800
-	0    -1   -1   0
+P 8350 4300
+F 0 "J2" V 8200 4550 50  0000 C CNN
+F 1 "433 mHz Transmitter" V 8100 4600 50  0000 C CNN
+F 2 "Connector_PinSocket_2.54mm:PinSocket_1x03_P2.54mm_Vertical" H 8350 4300 50  0001 C CNN
+F 3 "~" H 8350 4300 50  0001 C CNN
+	1    8350 4300
+	1    0    0    -1
 $EndComp
-Wire Wire Line
-	7550 3000 7550 2700
-Wire Wire Line
-	7450 3000 6450 3000
 NoConn ~ 7350 3500
 NoConn ~ 7200 3500
@@
 $EndComp
 Wire Wire Line
-	6300 2450 7300 2450
-Wire Wire Line
-	8850 2450 8850 4400
+	8850 2450 8850 3000
 Wire Wire Line
 	8850 5900 7300 5900
@@
 	6300 2450 6300 3500
 Wire Wire Line
-	7550 2700 7300 2700
-Wire Wire Line
-	7300 2700 7300 2450
-Connection ~ 7300 2450
-Wire Wire Line
-	7300 2450 8850 2450
-$Comp
-L 1-My~Parts:DHT11_Breakout J3
-U 1 1 5DA86315
-P 8350 4300
-F 0 "J3" H 8378 4326 50  0000 L CNN
-F 1 "DHT11_Breakout" H 8150 4100 50  0000 L CNN
-F 2 "Connector_PinSocket_2.54mm:PinSocket_1x03_P2.54mm_Vertical" H 8350 4300 50  0001 C CNN
-F 3 "~" H 8350 4300 50  0001 C CNN
-	1    8350 4300
-	1    0    0    -1
-$EndComp
-Wire Wire Line
 	6450 3500 6450 4200
 Wire Wire Line
 	6450 4200 8150 4200
-Wire Wire Line
-	8150 4300 7500 4300
-Wire Wire Line
-	7500 4300 7500 5050
-Wire Wire Line
-	8150 4400 8850 4400
-Connection ~ 8850 4400
-Wire Wire Line
-	8850 4400 8850 5900
 NoConn ~ 6600 5050
 NoConn ~ 5400 5050
 NoConn ~ 5700 5050
-Wire Wire Line
-	7650 3000 7650 3300
-Wire Wire Line
-	7650 3300 7500 3300
-Wire Wire Line
-	7500 3300 7500 3500
 NoConn ~ 7650 3500
 Wire Wire Line
@@
 	1    0    0    -1
 $EndComp
+$Comp
+L 1-My~Parts:DHT11_Breakout J3
+U 1 1 5DA86315
+P 7500 2800
+F 0 "J3" V 7438 2612 50  0000 R CNN
+F 1 "DHT11_Breakout" V 7347 2612 50  0000 R CNN
+F 2 "Connector_PinSocket_2.54mm:PinSocket_1x03_P2.54mm_Vertical" H 7500 2800 50  0001 C CNN
+F 3 "~" H 7500 2800 50  0001 C CNN
+	1    7500 2800
+	0    -1   -1   0
+$EndComp
+Wire Wire Line
+	6300 2450 8850 2450
+Wire Wire Line
+	7500 3000 7500 3500
+Wire Wire Line
+	7400 3000 6450 3000
+Wire Wire Line
+	7600 3000 8850 3000
+Connection ~ 8850 3000
+Wire Wire Line
+	7500 5050 7500 4400
+Wire Wire Line
+	7500 4400 8150 4400
+Wire Wire Line
+	8150 4300 8850 4300
+Wire Wire Line
+	8850 3000 8850 4300
+Connection ~ 8850 4300
+Wire Wire Line
+	8850 4300 8850 5900
 $EndSCHEMATC
